File: hardware/Can_EngineTranslator.kicad_pcb (KiCad board)
At the start: 2 copper layers, 72 x 63 mm, 63 parts, among them J1 ProgramerConnector, J2 CANcarConnector, J3 CANinverterConnector, J5 PowerOutputConnector, Q1 BSS138, SW1 SW_Push, U1 STM32F105RBTx, U2 LM2596S-5, U3 LM1117-3.3, U4 MCP2562-H-SN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

Commit message: PCB Fixed
Parts:
- added C21: CP_Small, Capacitor_SMD:C_1206_3216Metric, F.Cu at (74.3, 50.2)
- added C22: CP_Small, Capacitor_SMD:C_1206_3216Metric, F.Cu at (74.3, 54.8)
- added C23: 100nF, Capacitor_SMD:C_0805_2012Metric, F.Cu at (126.4, 71.8)
- added C24: 100nF, Capacitor_SMD:C_0805_2012Metric, F.Cu at (110.5, 58.8)
- R1: value 10k -> 100k
- R2: value 100k -> 10k
- moved D7 17.1 mm to (72.4, 40.7), turned to 180 degrees
- moved D8 14.5 mm to (72.4, 44.5), turned to 180 degrees
- moved C11 6.66 mm to (75.1, 57.1), turned to 180 degrees
- moved C14 6.07 mm to (110.4, 41.3), turned to 90 degrees
- moved C10 5.86 mm to (81.2, 57.7)
- moved D9 5.58 mm to (87.6, 57.6)
- moved C12 5.36 mm to (120.1, 48.7), turned to 270 degrees
- moved J2 3.83 mm to (66.5, 87.3)
- moved J3 3.83 mm to (66.5, 75.7)
- moved F1 3.59 mm to (72.6, 36.2), turned to 180 degrees
- moved J5 3.45 mm to (66.7, 45.0)
- moved FB1 3.16 mm to (78.0, 51.2), turned to 270 degrees
- moved U2 2.69 mm to (87.6, 43.4)
- moved C17 2.02 mm to (74.3, 48.0), turned to 180 degrees
- moved C18 1.21 mm to (74.3, 52.5)
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Connections:
- D7 pad 1: Net-(C10-Pad1) -> Net-(C17-Pad1)
- D8 pad 1: Net-(C10-Pad1) -> Net-(C17-Pad1)
- FB1 pad 1: Net-(C10-Pad1) -> Net-(C17-Pad1)
- FB1 pad 2: Net-(C17-Pad1) -> Net-(C10-Pad1)
Routing:
- net +5V: track 133.7 -> 101.4 mm
- net Net-(D9-Pad1): track 40.0 -> 23.1 mm
- net SW_GND: track 51.5 -> 40.7 mm, vias 26 -> 71
- net Net-(C17-Pad1): track 8.72 -> 17.5 mm
- net Net-(C10-Pad1): track 26.3 -> 20.7 mm
- net CANcar_L: track 17.8 -> 21.6 mm
- net CANcar_H: track 24.3 -> 28.1 mm
- net CANinverter_L: track 16.4 -> 20.2 mm
- net CANinverter_H: track 21.3 -> 25.1 mm
- net VCC: track 6.93 -> 6.16 mm

Commit message: Add files via upload
Parts:
- added G***: LOGO, Logos:SignatureBox25mm, B.Cu at (94.7, 41.9)
Other:
- board text added: "M. Przydatek S. Sambor"
- board text removed: "PUT Motorsport CAN translator M. Przydatek S. Sambor"
